Commit message: Adjust package name to match git

File: models/block.urdf.xacro (robot description, xacro)
@@ -5,5 +5,5 @@
   <xacro:macro name="block" params="block_number block_type">
     <!-- Parameters for reusability -->
-    <xacro:property name="mesh_path" value="$(find ros2_ur5_interface)/models/meshes/${block_type}.stl" />
+    <xacro:property name="mesh_path" value="$(find speed_controlled_ros2_ur5_interface)/models/meshes/${block_type}.stl" />
     <xacro:property name="mass" value="0.01" />
     <xacro:property name="ixx" value="3.604e-6" />

File: models/desk.urdf.xacro (robot description, xacro)
@@ -34,5 +34,5 @@
       <origin xyz="0 0 0" rpy="0 0 0" />
       <geometry>
-        <mesh filename="file://$(find ros2_ur5_interface)/models/meshes/desk.stl" scale="0.001 0.001 0.001" />
+        <mesh filename="file://$(find speed_controlled_ros2_ur5_interface)/models/meshes/desk.stl" scale="0.001 0.001 0.001" />
       </geometry>
       <material name="grey_material">

File: models/soft_robotics_gripper.xacro (robot description, xacro)
@@ -17,5 +17,5 @@
         <origin rpy="0 0 0" xyz="0 0 -0.0095" />
         <geometry>
-          <mesh filename="file://$(find ros2_ur5_interface)/models/meshes/base.stl"/>
+          <mesh filename="file://$(find speed_controlled_ros2_ur5_interface)/models/meshes/base.stl"/>
         </geometry>
         <material name="Grey" />
@@ -24,5 +24,5 @@
         <origin rpy="0 0 0" xyz="0 0 -0.0095" />
         <geometry>
-          <mesh filename="file://$(find ros2_ur5_interface)/models/meshes/base.stl"/>
+          <mesh filename="file://$(find speed_controlled_ros2_ur5_interface)/models/meshes/base.stl"/>
         </geometry>
       </collision>
@@ -44,12 +44,12 @@
         <origin rpy="0 0 0" xyz="0 0 0" />
         <geometry>
-          <mesh filename="file://$(find ros2_ur5_interface)/models/meshes/link1.stl"/>
-        </geometry>
-        <material name="Blue" />
-      </visual>
-      <collision>
-        <origin rpy="0 0 0" xyz="0 0 0" />
-        <geometry>
-          <mesh filename="file://$(find ros2_ur5_interface)/models/meshes/link1.stl"/>
+          <mesh filename="file://$(find speed_controlled_ros2_ur5_interface)/models/meshes/link1.stl"/>
+        </geometry>
+        <material name="Blue" />
+      </visual>
+      <collision>
+        <origin rpy="0 0 0" xyz="0 0 0" />
+        <geometry>
+          <mesh filename="file://$(find speed_controlled_ros2_ur5_interface)/models/meshes/link1.stl"/>
         </geometry>
       </collision>
@@ -71,12 +71,12 @@
         <origin rpy="0 0 0" xyz="0 0 0" />
         <geometry>
-          <mesh filename="file://$(find ros2_ur5_interface)/models/meshes/link1.stl"/>
-        </geometry>
-        <material name="Blue" />
-      </visual>
-      <collision>
-        <origin rpy="0 0 0" xyz="0 0 0" />
-        <geometry>
-          <mesh filename="file://$(find ros2_ur5_interface)/models/meshes/link1.stl"/>
+          <mesh filename="file://$(find speed_controlled_ros2_ur5_interface)/models/meshes/link1.stl"/>
+        </geometry>
+        <material name="Blue" />
+      </visual>
+      <collision>
+        <origin rpy="0 0 0" xyz="0 0 0" />
+        <geometry>
+          <mesh filename="file://$(find speed_controlled_ros2_ur5_interface)/models/meshes/link1.stl"/>
         </geometry>
       </collision>
@@ -95,11 +95,11 @@
       <visual>
         <geometry>
-          <mesh filename="file://$(find ros2_ur5_interface)/models/meshes/link2.stl"/>
-        </geometry>
-        <material name="Blue" />
-      </visual>
-      <collision>
-        <geometry>
-          <mesh filename="file://$(find ros2_ur5_interface)/models/meshes/link2.stl"/>
+          <mesh filename="file://$(find speed_controlled_ros2_ur5_interface)/models/meshes/link2.stl"/>
+        </geometry>
+        <material name="Blue" />
+      </visual>
+      <collision>
+        <geometry>
+          <mesh filename="file://$(find speed_controlled_ros2_ur5_interface)/models/meshes/link2.stl"/>
         </geometry>
       </collision>
@@ -118,11 +118,11 @@
       <visual>
         <geometry>
-          <mesh filename="file://$(find ros2_ur5_interface)/models/meshes/link2.stl"/>
-        </geometry>
-        <material name="Blue" />
-      </visual>
-      <collision>
-        <geometry>
-          <mesh filename="file://$(find ros2_ur5_interface)/models/meshes/link2.stl"/>
+          <mesh filename="file://$(find speed_controlled_ros2_ur5_interface)/models/meshes/link2.stl"/>
+        </geometry>
+        <material name="Blue" />
+      </visual>
+      <collision>
+        <geometry>
+          <mesh filename="file://$(find speed_controlled_ros2_ur5_interface)/models/meshes/link2.stl"/>
         </geometry>
       </collision>

File: models/ur_gz.urdf.xacro (robot description, xacro)
@@ -6,5 +6,5 @@
   <xacro:include filename="$(find ur_description)/urdf/ur_macro.xacro"/>
   <xacro:include filename="soft_robotics_gripper.xacro"/>
-  <xacro:include filename="$(find ros2_ur5_interface)/models/ur_gz.ros2_control.xacro" />
+  <xacro:include filename="$(find speed_controlled_ros2_ur5_interface)/models/ur_gz.ros2_control.xacro" />
   <!-- possible 'ur_type' values: ur3, ur3e, ur5, ur5e, ur10, ur10e, ur16e, ur20, ur30 -->
   <!-- the default value should raise an error in case this was called without defining the type -->
